Commit message: arm_flex_linkの慣性モーメントのixxの値だけ大きすぎたので修正
SolidWorksで大体の値を計算して1/1000した

File: urdf/arm_v0/arm.urdf.xacro (robot description, xacro)
@@ -67,5 +67,5 @@
                 <mass value="1.339295"/>
                 <origin xyz="0.000632 0.006404 0.118529"/>
-                <inertia ixx="7.528" ixy="-0.000020284207" ixz="-0.000022947194"
+                <inertia ixx="0.007528" ixy="-0.000020284207" ixz="-0.000022947194"
                     iyy="0.007102" iyz="-0.000091796075" izz="0.001552"/>
             </inertial>
