Commit message: シミュレーションの安定化のために摩擦設定追加

File: urdf/base_v2/base.urdf.xacro (robot description, xacro)
@@ -49,5 +49,5 @@
             <parent link="${parent}" />
             <child link="${prefix}_${suffix}_drive_wheel_link" />
-            <dynamics damping="1.0"/>
+            <dynamics damping="1.0" friction="1.0"/>
         </joint>
         <link name="${prefix}_${suffix}_drive_wheel_link">
@@ -197,5 +197,5 @@
             <parent link="${prefix}_link" />
             <child link="${prefix}_roll_link" />
-            <dynamics damping="0.7"/>
+            <dynamics damping="1.0" friction="1.0"/>
         </joint>
         <link name="${prefix}_roll_link">
